File: custom-espc5-board/Custom-ESPC5.kicad_pcb (KiCad board)
At the start: 2 copper layers, 0 parts

Commit message: finish schem, start board work
Parts:
- added C1: 0.1µ, Capacitor_SMD:C_0402_1005Metric, F.Cu at (178.9, 117.8)
- added C14: 0.012µF, Capacitor_SMD:C_0402_1005Metric, F.Cu at (178.9, 131.6)
- added C2: 1µ, Capacitor_SMD:C_0402_1005Metric, F.Cu at (178.9, 119.8)
- added C3: 0.1µ, Capacitor_SMD:C_0402_1005Metric, F.Cu at (178.9, 121.8)
- added C4: 0.1µ, Capacitor_SMD:C_0402_1005Metric, F.Cu at (178.9, 123.7)
- added C5: 0.1uF, Capacitor_SMD:C_0402_1005Metric, F.Cu at (178.9, 125.7)
- added C6: 10µF, Capacitor_SMD:C_0402_1005Metric, F.Cu at (178.9, 127.7)
- added C9: 47uF, Capacitor_SMD:C_0402_1005Metric, F.Cu at (178.9, 129.6)
- added D1: D, Diode_SMD:USC-TOS, F.Cu at (151.4, 130.4)
- added D2: SP0503BAHT, Package_TO_SOT_SMD:SOT-143, F.Cu at (173.6, 129.7)
- added J1: Screw_Terminal_01x02, TerminalBlock:TerminalBlock_MaiXu_MX126-5.0-02P_1x02_P5.00mm, F.Cu at (152.9, 123.8)
- added J10: Barrel_Jack, Connector_BarrelJack:BarrelJack_CUI_PJ-063AH_Horizontal, F.Cu at (172.3, 93.7)
- added J12: Conn_01x05, Connector_JST:JST_XH_S5B-XH-A-1_1x05_P2.50mm_Horizontal, F.Cu at (152.3, 96.6)
- added J13: Conn_01x05, Connector_JST:JST_XH_S5B-XH-A-1_1x05_P2.50mm_Horizontal, F.Cu at (152.3, 110.1)
- added J2: Conn_01x03, Connector_JST:JST_XH_S3B-XH-A-1_1x03_P2.50mm_Horizontal, F.Cu at (131.6, 83.0)
- added J3: Conn_01x03, Connector_JST:JST_XH_S3B-XH-A-1_1x03_P2.50mm_Horizontal, F.Cu at (143.6, 83.0)
- added J4: USB_C_Receptacle_USB2.0_14P, Connector_USB:USB_C_Receptacle_HRO_TYPE-C-31-M-12, F.Cu at (171.6, 122.6)
- added J5: Conn_01x03, Connector_JST:JST_XH_S3B-XH-A-1_1x03_P2.50mm_Horizontal, F.Cu at (155.5, 83.0)
- added J6: Screw_Terminal_01x03, TerminalBlock:TerminalBlock_MaiXu_MX126-5.0-03P_1x03_P5.00mm, F.Cu at (169.8, 111.7)
- added JP1: Jumper_2_Open, Connector_PinHeader_2.54mm:PinHeader_1x02_P2.54mm_Vertical, F.Cu at (140.3, 127.8)
- added JP2: Jumper_2_Open, Connector_PinHeader_2.54mm:PinHeader_1x02_P2.54mm_Vertical, F.Cu at (144.9, 127.8)
- added R1: 910, Resistor_SMD:R_0402_1005Metric, F.Cu at (139.4, 116.6)
- added R15: 5.1kΩ, Resistor_SMD:R_0402_1005Metric, F.Cu at (142.3, 124.5)
- added R16: 10k, Resistor_SMD:R_0402_1005Metric, F.Cu at (145.2, 116.6)
- added R17: 10k, Resistor_SMD:R_0402_1005Metric, F.Cu at (145.2, 118.6)
- added R18: 120, Resistor_SMD:R_0402_1005Metric, F.Cu at (145.2, 120.6)
- added R2: 270, Resistor_SMD:R_0402_1005Metric, F.Cu at (139.4, 118.6)
- added R3: 5.1k, Resistor_SMD:R_0402_1005Metric, F.Cu at (139.4, 120.6)
- added R4: 5.1k, Resistor_SMD:R_0402_1005Metric, F.Cu at (139.4, 122.5)
- added R5: 22.1k, Resistor_SMD:R_0402_1005Metric, F.Cu at (139.4, 124.5)
- added R6: 47.5k, Resistor_SMD:R_0402_1005Metric, F.Cu at (142.3, 116.6)
- added R7: 10k, Resistor_SMD:R_0402_1005Metric, F.Cu at (142.3, 118.6)
- added R8: 10k, Resistor_SMD:R_0402_1005Metric, F.Cu at (142.3, 120.6)
- added R9: 10k, Resistor_SMD:R_0402_1005Metric, F.Cu at (142.3, 122.5)
- added SW1: SW_Nidec_CAS-120A1, Button_Switch_SMD:Nidec_Copal_CAS-120A, F.Cu at (166.7, 88.2)
- added SW3: CK_KMS2xxG, Button_Switch_SMD:SW_SPST_CK_KMS2xxGP, F.Cu at (175.7, 87.8)
- added U1: ESP32-C5-WROOM-1U, PCM_Espressif:ESP32-C5-WROOM-1U, F.Cu at (138.2, 103.6)
- added U10: CP2102N-Axx-xQFN28, Package_DFN_QFN:QFN-28-1EP_5x5mm_P0.5mm_EP3.35x3.35mm, F.Cu at (176.4, 81.7)
- added U12: LM3940, Package_TO_SOT_SMD:SOT-223-3_TabPin2, F.Cu at (133.1, 128.1)
- added U2: LM317DCYR, Package_TO_SOT_SMD:SOT-223-3_TabPin2, F.Cu at (133.1, 119.8)
- added U5: INA219AxD, Package_SO:SOIC-8_3.9x4.9mm_P1.27mm, F.Cu at (168.2, 81.5)
- added U9: TJA1051TK-3, Package_SON:HVSON-8-1EP_3x3mm_P0.65mm_EP1.6x2.4mm, F.Cu at (168.8, 129.6)
