File: custom-espc5-board/Custom-ESPC5.kicad_pcb (KiCad board)
At the start: 4 copper layers, 64.8 x 62.3 mm, 44 parts, among them J1 Screw_Terminal_01x02, J10 Barrel_Jack, J12 Conn_01x05, J13 Conn_01x05, J2 Conn_01x03, J3 Conn_01x03, J4 USB_C_Receptacle_USB2.0_14P, J5 Conn_01x03, J6 Screw_Terminal_01x03, SW1 SW_Nidec_CAS-120A1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

Commit message: custom board preliminary complete
Parts:
- removed the ? at (51.1, 83.8)
- added ?: , , F.Cu at (51.5, 83.9)
- added ?: , , F.Cu at (108.9, 83.9)
- added R11: 10k, Resistor_SMD:R_0402_1005Metric, F.Cu at (83.6, 87.7)
- added SW2: SW_Push, Button_Switch_SMD:SW_SPST_PTS810, F.Cu at (69.4, 84.0)
- SW3: value CK_KMS2xxG -> SW_Push; footprint Button_Switch_SMD:SW_SPST_CK_KMS2xxGP -> Button_Switch_SMD:SW_SPST_PTS810
- moved R15 55.3 mm to (62.1, 84.7), turned to 90 degrees
- moved C14 55.1 mm to (63.4, 84.6), turned to -90 degrees
- moved R16 55.0 mm to (64.5, 84.6), turned to 90 degrees
- moved SW3 46.3 mm to (81.4, 84.0), turned to 0 degrees
- moved U9 6.51 mm to (83.1, 122.4)
- moved R17 5.37 mm to (86.6, 122.4)
- moved J6 4.58 mm to (88.7, 138.1), turned to 0 degrees
- moved J1 2.89 mm to (99.1, 138.1), turned to 0 degrees
- moved R18 1.92 mm to (89.2, 132.4), turned to 0 degrees
- moved SW1 0.80 mm to (90.8, 126.7), turned to 90 degrees
- moved ? 0.47 mm to (51.5, 138.6)
- moved ? 0.15 mm to (108.9, 138.6)
Connections:
- SW3 pad 2: Net-(R16-Pad2) -> Net-(R11-Pad2)
- U1 pad 15: unconnected-(U1-GPIO28-Pad15) -> /GPIO28
Routing:
- net /CHIP_PU: track 68.3 -> 15.9 mm, vias 0 -> 2
- net /GPIO28: track 0.00 -> 23.5 mm, vias 0 -> 2
- net GND: track 80.5 -> 91.5 mm, vias 33 -> 35
- net Net-(J6-Pin_3): track 18.9 -> 27.0 mm, vias 0 -> 2
- net Net-(R11-Pad2): track 0.00 -> 6.99 mm
- net Net-(J6-Pin_1): track 21.9 -> 16.5 mm
- net Net-(R16-Pad2): track 11.5 -> 7.50 mm
- net +5V: track 20.4 -> 24.1 mm
- net Net-(SW1-B): track 4.94 -> 7.33 mm
- net Net-(J1-Pin_1): track 7.87 -> 6.43 mm
- net Net-(U9-S): track 1.58 -> 2.91 mm
- net /CAN RX: track 14.7 -> 15.8 mm, vias 2 -> 0
- net +3.3V: vias 7 -> 6
Other:
- board text added: "BOOT"

Commit message: Increase density
Parts:
- moved J5 58.6 mm to (104.5, 124.8), turned to 90 degrees
- moved J13 11.3 mm to (56.5, 92.5)
- moved J12 10.1 mm to (56.5, 110.2)
- moved R8 7.60 mm to (94.8, 118.6)
- moved R9 7.60 mm to (93.5, 118.6)
- moved U5 7.60 mm to (93.0, 123.6)
- moved SW1 6.89 mm to (85.8, 121.8)
- moved J1 5.97 mm to (96.7, 132.6)
- moved J6 5.92 mm to (86.6, 132.6)
- moved U9 5.87 mm to (79.7, 117.6)
- moved R17 5.87 mm to (83.2, 117.6)
- moved J2 5.63 mm to (61.8, 129.2)
- moved R18 5.59 mm to (86.9, 127.3)
- moved J3 5.47 mm to (74.8, 129.2)
- moved ? 5.30 mm to (51.4, 133.2)
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Routing:
- net /WS2812: track 13.0 -> 47.1 mm, vias 0 -> 1
- net +3.3V: track 157.7 -> 185.9 mm, vias 6 -> 4
- net /IDX1: track 34.2 -> 20.8 mm
- net /IDX2: track 36.2 -> 24.5 mm
- net /SIG1: track 42.2 -> 34.4 mm, vias 0 -> 1
- net /A1: track 29.4 -> 21.7 mm
- net /I2C SDA: track 43.4 -> 35.9 mm
- net /I2C SCL: track 43.0 -> 36.1 mm
- net /B2: track 33.8 -> 27.6 mm, vias 3 -> 0
- net /SIG2: track 46.8 -> 41.1 mm, vias 0 -> 1
- net /A2: track 39.7 -> 34.7 mm, vias 2 -> 0
- net GND: track 91.5 -> 87.4 mm
- net Net-(J6-Pin_3): track 27.0 -> 23.4 mm
- net /CAN TX: track 17.3 -> 14.0 mm
- net /B1: track 33.2 -> 30.7 mm
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Other:
- board size 64.8 x 62.3 mm -> 64.8 x 57 mm

Commit message: fixed schematic changes
fixed schematic changes like master austin said
Parts:
- added C10: 1µ, Capacitor_SMD:C_0402_1005Metric, F.Cu at (123.5, 129.1)
- added C11: 0.1µ, Capacitor_SMD:C_0402_1005Metric, F.Cu at (123.5, 131.1)
- added C12: 1µ, Capacitor_SMD:C_0402_1005Metric, F.Cu at (123.5, 133.0)
- added C13: 0.1µ, Capacitor_SMD:C_0402_1005Metric, F.Cu at (123.5, 135.0)
- added C15: 1µ, Capacitor_SMD:C_0402_1005Metric, F.Cu at (132.5, 129.0)
- added C16: 0.1µ, Capacitor_SMD:C_0402_1005Metric, F.Cu at (132.5, 131.0)
- added C8: NC, Capacitor_SMD:C_0402_1005Metric, F.Cu at (137.5, 110.0)
- added C9: 0.1µ, Capacitor_SMD:C_0402_1005Metric, F.Cu at (123.5, 127.1)
- added Q1: BC847BDW1, Package_TO_SOT_SMD:SOT-363_SC-70-6, F.Cu at (125.1, 112.3)
- added R10: R, Resistor_SMD:R_0402_1005Metric, F.Cu at (134.5, 110.0)
- added R12: R, Resistor_SMD:R_0402_1005Metric, F.Cu at (134.5, 112.0)
- added R13: R, Resistor_SMD:R_0402_1005Metric, F.Cu at (134.5, 114.0)
- added R14: 10K, Resistor_SMD:R_0402_1005Metric, F.Cu at (134.5, 116.0)
- added R19: 10K, Resistor_SMD:R_0402_1005Metric, F.Cu at (134.5, 118.0)
- added R20: 10k, Resistor_SMD:R_0402_1005Metric, F.Cu at (129.6, 129.0)
- added R21: 10k, Resistor_SMD:R_0402_1005Metric, F.Cu at (129.6, 131.0)
- R1: value 910 -> 750
Connections:
- J1 pad 2: GND -> Net-(J1-Pin_2)
- U5 pad 3: /I2C SDA -> Net-(U5-SDA)
- U5 pad 4: /I2C SCL -> Net-(U5-SCL)
- U5 pad 7: GND -> Net-(J1-Pin_2)
Routing:
- net Net-(J1-Pin_2): track 0.00 -> 2.63 mm, vias 0 -> 1
- net GND: track 87.4 -> 84.8 mm, vias 35 -> 34
