File: custom-espc5-board/Custom-ESPC5.kicad_sch (KiCad schematic)
At the start: 0 parts

Commit message: finish schem, start board work
Parts:
- added C1, C3, C4: 0.1µ, Capacitor_SMD:C_0402_1005Metric, symbol Device:C
- added C14: 0.012µF, Capacitor_SMD:C_0402_1005Metric, symbol Device:C
- added C2: 1µ, Capacitor_SMD:C_0402_1005Metric, symbol Device:C
- added C5: 0.1uF, Capacitor_SMD:C_0402_1005Metric, symbol Device:C
- added C6: 10µF, Capacitor_SMD:C_0402_1005Metric, symbol Device:C
- added C9: 47uF, Capacitor_SMD:C_0402_1005Metric, symbol Device:C
- added D1: D, Diode_SMD:USC-TOS, symbol Device:D
- added D2: SP0503BAHT, Package_TO_SOT_SMD:SOT-143, symbol Power_Protection:SP0503BAHT
- added J1: Screw_Terminal_01x02, TerminalBlock:TerminalBlock_MaiXu_MX126-5.0-02P_1x02_P5.00mm, symbol Connector:Screw_Terminal_01x02
- added J10: Barrel_Jack, Connector_BarrelJack:BarrelJack_CUI_PJ-063AH_Horizontal, symbol Connector:Barrel_Jack
- added J12, J13: Conn_01x05, Connector_JST:JST_XH_S5B-XH-A-1_1x05_P2.50mm_Horizontal, symbol Connector_Generic:Conn_01x05
- added J2, J3, J5: Conn_01x03, Connector_JST:JST_XH_S3B-XH-A-1_1x03_P2.50mm_Horizontal, symbol Connector_Generic:Conn_01x03
- added J4: USB_C_Receptacle_USB2.0_14P, Connector_USB:USB_C_Receptacle_HRO_TYPE-C-31-M-12, symbol Connector:USB_C_Receptacle_USB2.0_14P
- added J6: Screw_Terminal_01x03, TerminalBlock:TerminalBlock_MaiXu_MX126-5.0-03P_1x03_P5.00mm, symbol Connector:Screw_Terminal_01x03
- added JP1, JP2: Jumper_2_Open, Connector_PinHeader_2.54mm:PinHeader_1x02_P2.54mm_Vertical, symbol Jumper:Jumper_2_Open
- added R1: 910, Resistor_SMD:R_0402_1005Metric, symbol Device:R
- added R15: 5.1kΩ, Resistor_SMD:R_0402_1005Metric, symbol Device:R
- added R16, R17, R7, R8, R9: 10k, Resistor_SMD:R_0402_1005Metric, symbol Device:R
- added R18: 120, Resistor_SMD:R_0402_1005Metric, symbol Device:R
- added R2: 270, Resistor_SMD:R_0402_1005Metric, symbol Device:R
- added R3, R4: 5.1k, Resistor_SMD:R_0402_1005Metric, symbol Device:R
- added R5: 22.1k, Resistor_SMD:R_0402_1005Metric, symbol Device:R
- added R6: 47.5k, Resistor_SMD:R_0402_1005Metric, symbol Device:R
- added SW1: SW_Nidec_CAS-120A1, Button_Switch_SMD:Nidec_Copal_CAS-120A, symbol Switch:SW_Nidec_CAS-120A1
- added SW3: CK_KMS2xxG, Button_Switch_SMD:SW_SPST_CK_KMS2xxGP, symbol Switch:CK_KMS2xxG
- added U1: ESP32-C5-WROOM-1U, PCM_Espressif:ESP32-C5-WROOM-1U, symbol PCM_Espressif:ESP32-C5-WROOM-1U
- added U10: CP2102N-Axx-xQFN28, Package_DFN_QFN:QFN-28-1EP_5x5mm_P0.5mm_EP3.35x3.35mm, symbol Interface_USB:CP2102N-Axx-xQFN28
- added U12: LM3940, Package_TO_SOT_SMD:SOT-223-3_TabPin2, symbol Regulator_Linear:LM3940
- added U2: LM317DCYR, Package_TO_SOT_SMD:SOT-223-3_TabPin2, symbol Regulator_Linear:LM317_TO-263
- added U5: INA219AxD, Package_SO:SOIC-8_3.9x4.9mm_P1.27mm, symbol Sensor_Energy:INA219AxD
- added U9: TJA1051TK-3, Package_SON:HVSON-8-1EP_3x3mm_P0.65mm_EP1.6x2.4mm, symbol Interface_CAN_LIN:TJA1051TK-3
Connections:
- new net: J1.1 (Pin_1), U5.8 (IN+)
- new net: C5.1, C6.1, D2.2 (K), J4.A4 (VBUS), J4.A9 (VBUS), J4.B4 (VBUS), J4.B9 (VBUS), R5.1, U10.7 (VREGIN)
- new net: C2.1, D1.2 (A), R2.2, U2.2 (VO)
- new net: D2.3 (K), J4.A7 (D-), J4.B7 (D-), U10.5 (D-)
- new net: D2.4 (K), J4.A6 (D+), J4.B6 (D+), U10.4 (D+)
- new net: R16.2, SW3.2
- new net: J4.A5 (CC1), R4.1
- new net: J6.1 (Pin_1), R18.1, U9.7 (CANH)
- new net: R18.2, SW1.2 (B)
- new net: R1.2, R2.1, U2.1 (ADJ)
- new net: R5.2, R6.1, U10.8 (VBUS)
- new net: R7.2, U10.9 (~{RST})
- new net: R17.1, U9.8 (S)
- new net: J4.B5 (CC2), R3.1
- new net: J6.3 (Pin_3), SW1.3 (A), U9.6 (CANL)
- new net: JP2.1 (A), R9.1, U5.2 (A0)
- new net: JP1.1 (A), R8.1, U5.1 (A1)
- new net: C1.1, J10.1, U2.3 (VI)
- new net +3.3V: C9.1, J12.1 (Pin_1), J13.1 (Pin_1), J2.1 (Pin_1), J3.1 (Pin_1), J5.1 (Pin_1), R15.1, R7.1, U1.2 (3V3), U10.6 (VDD), U12.1 (OUT), U5.5 (VS), U9.5 (VIO)
- new net +3V3: JP1.2 (B), JP2.2 (B)
- new net +5V: D1.1 (K), U12.3 (IN), U9.3 (VCC)
- new net A1: J13.3 (Pin_3), U1.12 (GPIO10)
- new net A2: J12.3 (Pin_3), U1.21 (GPIO23)
- new net B1: J13.2 (Pin_2), U1.23 (GPIO24)
- new net B2: J12.2 (Pin_2), U1.5 (GPIO3)
- new net CAN RX: U1.16 (GPIO5), U9.4 (RXD)
- new net CAN TX: U1.17 (GPIO4), U9.1 (TXD)
- new net CHIP_PU: C14.2, R15.2, R16.1, U1.3 (EN/CHIP_PU)
- new net GND: C1.2, C14.1, C2.2, C3.2, C4.2, C5.2, C6.2, C9.2, D2.1 (A), J1.2 (Pin_2), J10.2, J12.5 (Pin_5), J13.5 (Pin_5), J2.3 (Pin_3), J3.3 (Pin_3), J4.A1 (GND), J4.A12 (GND), J4.B1 (GND), J4.B12 (GND), J5.3 (Pin_3), J6.2 (Pin_2), R1.1, R17.2, R3.2, R4.2, R6.2, R8.2, R9.2, SW3.1, SW3.SH (B), U1.1 (GND), U1.28 (GND), U1.29 (GND), U1.30 (GND), U1.32 (GND), U10.29 (GND), U10.3 (GND), U12.2 (GND), U5.6 (GND), U5.7 (IN-), U9.2 (GND), U9.9 (GND)
- new net I2C SCL: U1.9 (GPIO7), U5.4 (SCL)
- new net I2C SDA: U1.8 (GPIO6), U5.3 (SDA)
- new net IDX1: J13.4 (Pin_4), U1.10 (GPIO8)
- new net IDX2: J12.4 (Pin_4), U1.11 (GPIO9)
- new net SIG1: C3.1, J2.2 (Pin_2), U1.7 (GPIO1)
- new net SIG2: C4.1, J3.2 (Pin_2), U1.4 (GPIO2)
- new net UART DTR: U10.28 (~{DTR})
- new net UART RTS: U10.24 (~{RTS})
- new net UART RX: U10.25 (RXD)
- new net UART TX: U10.26 (TXD)
- new net WS2812: J5.2 (Pin_2), U1.6 (GPIO0)
- no-connect marks 0 -> 17
Other:
- note added: "5V -> 3.3V Regulator"
- note added: "Analog"
- note added: "Analog 1"
- note added: "Analog 2"
- note added: "CAN"
- note added: "Encoder 1"
- note added: "Encoder 2"
- note added: "Forward voltage drop: 0.1 V @ 10mA 0.22V @ 100 mA 0.34 V @ 1 A"
- note added: "I_Adj = 50 µA"
- note added: "PDP Step-Down"
- note added: "PDP-V"
- note added: "Quadrature Encoders"
- note added: "Reset Switch"
- note added: "Spike"
- note added: "USB Serial"
- note added: "VO = 1.25 * (1 + R1/R2) + I_Adj * R2 = 5.5 V"
- note added: "Vcc"
- note added: "Voltage Sensor"
- note added: "WS2812 LEDs"
- note added: "~15.2 V"

Commit message: board layout
Parts:
- removed U10: CP2102N-Axx-xQFN28, Package_DFN_QFN:QFN-28-1EP_5x5mm_P0.5mm_EP3.35x3.35mm, symbol Interface_USB:CP2102N-Axx-xQFN28
- added D3: D, Diode_SMD:USC-TOS, symbol Device:D
- added U3: CP2102N-Axx-xQFN24, Package_DFN_QFN:QFN-24-1EP_4x4mm_P0.5mm_EP2.6x2.6mm, symbol Interface_USB:CP2102N-Axx-xQFN24
- R1: value 910 -> 430
- R2: value 270 -> 240
Connections:
- net +3.3V: now also D1.1 (K), D3.1 (K), U3.5 (VIO), U3.6 (VDD); no longer C9.1, U12.1 (OUT)
- net +5V: no longer D1.1 (K), U12.3 (IN)
- net GND: now also U3.2 (GND), U3.25 (GND)
- net UART DTR: now also U3.23 (~{DTR})
- net UART RTS: now also U3.19 (~{RTS})
- net UART RX: now also U3.20 (RXD)
- net UART TX: now also U3.21 (TXD)
- net at C5.1, C6.1, D2.2 (K)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: now also U12.3 (IN), U3.7 (VREGIN)
- net at D2.3 (K), J4.A7 (D-), J4.B7 (D-): now also U3.4 (D-)
- net at D2.4 (K), J4.A6 (D+), J4.B6 (D+): now also U3.3 (D+)
- net at R5.2, R6.1: now also U3.8 (VBUS)
- net at R7.2: now also U3.9 (~{RST})
- new net: C9.1, D3.2 (A), U12.1 (OUT)
- no-connect marks 17 -> 11
Other:
- note added: "USB Stackup"
- note added: "VO = 1.25 * (1 + R1/R2) + I_Adj * R2 = 3.5 V"
- note added: "Wolfwood"
- note removed: "5V -> 3.3V Regulator"
- note removed: "Spike"
- note removed: "USB Serial"
- note removed: "VO = 1.25 * (1 + R1/R2) + I_Adj * R2 = 5.5 V"
- moved on the sheet: C5, C6, C9, D2, J4, R3, R4, R5, R6, R7, U12

Commit message: Finish preliminary board tracings (NOT COMPLETE)
Parts:
- removed C9: 47uF, Capacitor_SMD:C_0402_1005Metric, symbol Device:C
- removed D3: D, Diode_SMD:USC-TOS, symbol Device:D
- removed JP1, JP2: Jumper_2_Open, Connector_PinHeader_2.54mm:PinHeader_1x02_P2.54mm_Vertical, symbol Jumper:Jumper_2_Open
- removed U12: LM3940, Package_TO_SOT_SMD:SOT-223-3_TabPin2, symbol Regulator_Linear:LM3940
- added C7: 47uF, Capacitor_SMD:C_0402_1005Metric, symbol Device:C
- added D4: D, Diode_SMD:USC-TOS, symbol Device:D
- added U4: LM3940, Package_TO_SOT_SMD:SOT-223-3_TabPin2, symbol Regulator_Linear:LM3940
- J1: footprint TerminalBlock:TerminalBlock_MaiXu_MX126-5.0-02P_1x02_P5.00mm -> TerminalBlock:TerminalBlock_Xinya_XY308-2.54-2P_1x02_P2.54mm_Horizontal
- J6: footprint TerminalBlock:TerminalBlock_MaiXu_MX126-5.0-03P_1x03_P5.00mm -> TerminalBlock:TerminalBlock_Xinya_XY308-2.54-3P_1x03_P2.54mm_Horizontal
- R1: value 430 -> 910
Connections:
- net +3.3V: now also C7.1, U4.1 (OUT); no longer D1.1 (K)
- net +5V: now also D1.1 (K), D4.1 (K), U4.3 (IN)
- net GND: now also C7.2, U4.2 (GND)
- net UART RX: now also U1.24 (U0RXD/GPIO12), U3.21 (TXD); no longer U3.20 (RXD)
- net UART TX: now also U1.25 (U0TXD/GPIO11), U3.20 (RXD); no longer U3.21 (TXD)
- net at C5.1, C6.1, D2.2 (K)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: now also D4.2 (A)
Other:
- note added: "5V -> 3.3V"
- note added: "VO = 1.25 * (1 + R1/R2) + I_Adj * R2 = 5.5 V"
- note removed: "VO = 1.25 * (1 + R1/R2) + I_Adj * R2 = 3.5 V"
- moved on the sheet: J5, R7

Commit message: custom board preliminary complete
Parts:
- removed SW3: CK_KMS2xxG, Button_Switch_SMD:SW_SPST_CK_KMS2xxGP, symbol Switch:CK_KMS2xxG
- added R11: 10k, Resistor_SMD:R_0402_1005Metric, symbol Device:R
- added SW2, SW3: SW_Push, Button_Switch_SMD:SW_SPST_EVQPE1, symbol Switch:SW_Push
Connections:
- net GND: now also SW2.1, SW3.1
- net at R16.2: now also SW2.2
- net GPIO28: now reaches U1.15 (GPIO28)
- net GPIO28: now also R11.1
- new net: R11.2, SW3.2
Other:
- note added: "BOOT Switch"
- note added: "wolfwood"
- note removed: "Wolfwood"

Commit message: Increase density
Parts:
- SW2, SW3: footprint Button_Switch_SMD:SW_SPST_EVQPE1 -> Button_Switch_SMD:SW_SPST_PTS810
Other:
- note added: "wolfwood s3"
- note removed: "wolfwood"
Changed lines of the file:
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@@
 		)
 	)
-	(text "wolfwood\n"
+	(text "wolfwood s3\n"
 		(exclude_from_sim no)
 		(at 591.058 320.802 0)
@@
 			)
 		)
-		(property "Footprint" "Button_Switch_SMD:SW_SPST_EVQPE1"
+		(property "Footprint" "Button_Switch_SMD:SW_SPST_PTS810"
 			(at 528.32 299.72 0)
 			(effects
@@
 			)
 		)
-		(property "Footprint" "Button_Switch_SMD:SW_SPST_EVQPE1"
+		(property "Footprint" "Button_Switch_SMD:SW_SPST_PTS810"
 			(at 565.15 308.61 0)
 			(effects

Commit message: fix name
Other:
- note added: "wolfwood"
- note removed: "wolfwood s3"
Changed lines of the file:
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@@
 		)
 	)
-	(text "wolfwood s3\n"
+	(text "wolfwood"
 		(exclude_from_sim no)
-		(at 591.058 320.802 0)
+		(at 601.98 320.802 0)
 		(effects
 			(font

Commit message: Update Custom-ESPC5.kicad_sch
Made correction to lm317 circuit annotations
Other:
- note added: "VO = 1.25 * (1 + R1/R2) + I_Adj * R1 = 6.03 V"
- note removed: "VO = 1.25 * (1 + R1/R2) + I_Adj * R2 = 5.5 V"
Changed lines of the file:
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@@
 		)
 	)
-	(text "VO = 1.25 * (1 + R1/R2) + I_Adj * R2 = 5.5 V\n"
+	(text "VO = 1.25 * (1 + R1/R2) + I_Adj * R1 = 6.03 V\n"
 		(exclude_from_sim no)
 		(at 496.824 365.252 0)
@@
 			)
 		)
-		(property "Datasheet" "~"
+		(property "Datasheet" "https://www.ckswitches.com/media/1476/pts810.pdf"
 			(at 528.32 299.72 0)
 			(effects
@@
 			)
 		)
+		(property "Field5" ""
+			(at 528.32 304.8 0)
+			(effects
+				(font
+					(size 1.27 1.27)
+				)
+				(hide yes)
+			)
+		)
 		(pin "1"
 		)
@@
 			)
 		)
-		(property "Datasheet" "~"
+		(property "Datasheet" "https://www.ckswitches.com/media/1476/pts810.pdf"
 			(at 565.15 308.61 0)
 			(effects
