File: custom-esp32-S3-board/Custom-ESPC5.kicad_pcb (KiCad board)
At the start: 4 copper layers, 63.6 x 52.8 mm, 64 parts, among them J1 Screw_Terminal_01x02, J10 Barrel_Jack, J12 Conn_01x05, J13 Conn_01x05, J2 Conn_01x02_Pin, J3 Conn_01x02_Pin, J4 USB_C_Receptacle_USB2.0_14P, J5 Conn_01x03, J6 Screw_Terminal_01x03, J7 Conn_01x02_Pin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

Commit message: Final Edits
Generated gerbers
Parts:
- removed R11, R16: 10k, Resistor_SMD:R_0402_1005Metric
Connections:
- J1 pad 2: GND -> Net-(J1-Pin_2)
- SW2 pad 2: Net-(R16-Pad2) -> /CHIP_PU
- SW3 pad 2: Net-(R11-Pad2) -> /GPIO0
- U5 pad 7: GND -> Net-(J1-Pin_2)
Routing:
- net Net-(J1-Pin_2): track 0.00 -> 14.7 mm
- net /CHIP_PU: track 16.0 -> 29.3 mm
- net Net-(R16-Pad2): track 10.1 -> 0.00 mm
- net Net-(R11-Pad2): track 9.77 -> 0.00 mm
- net +3.3V: track 155.7 -> 152.3 mm
- net /A2: track 32.5 -> 30.6 mm, vias 5 -> 4
- net GND: track 99.3 -> 98.0 mm
- net unconnected-(U6-IO37-Pad30): vias 1 -> 0
- net /B2: vias 4 -> 2
Other:
- board text added: "120Ω"
- board text added: "ESP Quack Rev 1"
- board text added: "Roger Zhu Aryan Tadepalli"
- board text removed: "120 Ω"
- board text removed: "ESP Quack S3 DevBoard"
- board text removed: "RX"
- board text removed: "Roger Zhu Austen Yun"
- board text removed: "SCL"

Commit message: Edit silkscreen
Increased package size of C7 :(
Parts:
- C7: footprint Capacitor_SMD:C_0402_1005Metric -> Capacitor_SMD:C_0805_2012Metric
- moved C7 0.60 mm to (91.7, 110.0), turned to 0 degrees
Routing:
- net GND: track 98.0 -> 96.1 mm
- net +3.3V: track 152.3 -> 152.1 mm, vias 9 -> 10
Other:
- board text added: "NC"
- board text added: "Vbat"
- board text removed: "+"
- board text removed: "-"
Changed lines of the file:
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@@
 		(tags "TO-220-3 Vertical RM 2.54mm")
 		(property "Reference" "U4"
-			(at 2.625 -4.1 270)
+			(at 0.45 -4.15 270)
 			(layer "F.SilkS")
 			(effects
@@
 		(tags "2.4 GHz Wi-Fi and Bluetooth module")
 		(property "Reference" "U6"
-			(at -0.125 -7.35 0)
+			(at 0.05 -7.55 0)
 			(unlocked yes)
 			(layer "F.SilkS")
+			(hide yes)
 			(effects
 				(font
@@
 		(attr smd)
 		(fp_line
-			(start -9.2 -12.9)
-			(end -9.2 -6.7)
-			(stroke
-				(width 0.12)
-				(type solid)
-			)
-			(layer "F.SilkS")
-		)
-		(fp_line
-			(start -9.2 -12.9)
-			(end 9.2 -12.9)
-			(stroke
-				(width 0.12)
-				(type solid)
-			)
-			(layer "F.SilkS")
-		)
-		(fp_line
 			(start -9.2 11.95)
 			(end -9.2 12.95)
@@
 		)
 		(fp_line
-			(start 9.2 -12.9)
-			(end 9.2 -6.7)
-			(stroke
-				(width 0.12)
-				(type solid)
-			)
-			(layer "F.SilkS")
-		)
-		(fp_line
 			(start 9.2 12.95)
 			(end 7.7 12.95)
@@
 		)
 	)
-	(footprint "Capacitor_SMD:C_0402_1005Metric"
+	(footprint "Capacitor_SMD:C_0805_2012Metric"
 		(layer "F.Cu")
-		(at 92.1 109.55 -90)
-		(descr "Capacitor SMD 0402 (1005 Metric), square (rectangular) end terminal, IPC-7351 nominal, (Body size source: IPC-SM-782 page 76, https://www.pcb-3d.com/wordpress/wp-content/uploads/ipc-sm-782a_amendment_1_and_2.pdf), generated with kicad-footprint-generator")
+		(at 91.65 109.95)
+		(descr "Capacitor SMD 0805 (2012 Metric), square (rectangular) end terminal, IPC-7351 nominal, (Body size source: IPC-SM-782 page 76, https://www.pcb-3d.com/wordpress/wp-content/uploads/ipc-sm-782a_amendment_1_and_2.pdf, https://docs.google.com/spreadsheets/d/1BsfQQcO9C6DZCsRaXUlFlo91Tg2WpOkGARC1WS5S8t0/edit?usp=sharing), generated with kicad-footprint-generator")
 		(tags "capacitor")
 		(property "Reference" "C7"
-			(at 0.025 -0.95 90)
+			(at 0.75 -1.8 0)
 			(layer "F.SilkS")
 			(hide yes)
 			(effects
 				(font
-					(size 0.5 0.5)
-					(thickness 0.1)
-					(bold yes)
+					(size 1 1)
+					(thickness 0.15)
 				)
 			)
 		)
 		(property "Value" "47uF"
-			(at 0 1.16 90)
+			(at 0 1.68 0)
 			(layer "F.Fab")
 			(effects
@@
 		)
 		(property "Datasheet" "~"
-			(at 0 0 90)
+			(at 0 0 0)
 			(layer "F.Fab")
 			(hide yes)
@@
 		)
 		(property "Description" "Unpolarized capacitor"
-			(at 0 0 90)
+			(at 0 0 0)
 			(layer "F.Fab")
 			(hide yes)
@@
 		(attr smd)
 		(fp_line
-			(start -0.107836 0.36)
-			(end 0.107836 0.36)
+			(start -0.261252 -0.735)
+			(end 0.261252 -0.735)
 			(stroke
 				(width 0.12)
@@
 		)
 		(fp_line
-			(start -0.107836 -0.36)
-			(end 0.107836 -0.36)
+			(start -0.261252 0.735)
+			(end 0.261252 0.735)
 			(stroke
 				(width 0.12)
@@
 		)
 		(fp_rect
-			(start -0.91 -0.46)
-			(end 0.91 0.46)
+			(start -1.7 -0.98)
+			(end 1.7 0.98)
 			(stroke
 				(width 0.05)
@@
 		)
 		(fp_rect
-			(start -0.5 -0.25)
-			(end 0.5 0.25)
+			(start -1 -0.625)
+			(end 1 0.625)
 			(stroke
 				(width 0.1)
@@
 		)
 		(fp_text user "${REFERENCE}"
-			(at 0 0 90)
+			(at 0 0 0)
 			(layer "F.Fab")
 			(effects
 				(font
-					(size 0.25 0.25)
-					(thickness 0.04)
+					(size 0.5 0.5)
+					(thickness 0.08)
 				)
 			)
 		)
 		(pad "1" smd roundrect
-			(at -0.48 0 270)
-			(size 0.56 0.62)
+			(at -0.95 0)
+			(size 1 1.45)
 			(layers "F.Cu" "F.Mask" "F.Paste")
 			(roundrect_rratio 0.25)
@@
 		)
 		(pad "2" smd roundrect
-			(at 0.48 0 270)
-			(size 0.56 0.62)
+			(at 0.95 0)
+			(size 1 1.45)
 			(layers "F.Cu" "F.Mask" "F.Paste")
 			(roundrect_rratio 0.25)
@@
 		)
 		(embedded_fonts no)
-		(model "${KICAD9_3DMODEL_DIR}/Capacitor_SMD.3dshapes/C_0402_1005Metric.step"
+		(model "${KICAD9_3DMODEL_DIR}/Capacitor_SMD.3dshapes/C_0805_2012Metric.step"
 			(offset
 				(xyz 0 0 0)
@@
 		(tags "THT Terminal Block Xinya XY308-2.54-2P pitch 2.54mm size 5.58x6.5mm drill 1.2mm pad 2mm")
 		(property "Reference" "J1"
-			(at -1.26 5.4 0)
+			(at 5.39 2.4 0)
 			(layer "F.SilkS")
 			(effects
@@
 			(layer "F.SilkS")
 		)
-		(fp_poly
-			(pts
-				(xy 0 3.52) (xy 0.44 4.13) (xy -0.44 4.13)
-			)
-			(stroke
-				(width 0.12)
-				(type solid)
-			)
-			(fill yes)
-			(layer "F.SilkS")
-		)
 		(fp_rect
 			(start -2.02 -3.6)
@@
 	)
 	(gr_text "BOOT"
-		(at 90.925 82.425 0)
+		(at 96.85 85 0)
 		(layer "F.SilkS")
 		(effects
@@
 		)
 	)
-	(gr_text "+\n"
-		(at 74.65 120.425 0)
+	(gr_text "Vbat"
+		(at 77.55 129.2 0)
+		(layer "F.SilkS")
+		(effects
+			(font
+				(size 1 1)
+				(thickness 0.15)
+			)
+		)
+	)
+	(gr_text "NC"
+		(at 74.3 129.25 0)
 		(layer "F.SilkS")
 		(effects
@@
 	)
 	(gr_text "VSense\n"
-		(at 77.9 130.1 0)
+		(at 75.65 130.9 0)
 		(layer "F.SilkS")
 		(effects
@@
 	)
 	(gr_text "RESET"
-		(at 59.675 82.325 0)
+		(at 53.6 83.6 0)
 		(layer "F.SilkS")
 		(effects
@@
 		)
 	)
-	(gr_text "\n-\n"
-		(at 77.25 119.625 0)
-		(layer "F.SilkS")
-		(effects
-			(font
-				(size 1 1)
-				(thickness 0.15)
-			)
-		)
-	)
 	(gr_text "15V PDP IN"
 		(at 101.725 88.575 0)
@@
 	)
 	(segment
-		(start 97.75 106.6)
-		(end 97.75 106.1)
-		(width 0.2)
-		(layer "F.Cu")
-		(net 2)
-	)
-	(segment
 		(start 70.15 116.3)
 		(end 70.15 117.395)
@@
 	)
 	(segment
-		(start 97.75 107.1)
-		(end 98.178298 107.1)
-		(width 0.2)
-		(layer "F.Cu")
-		(net 2)
-	)
-	(segment
 		(start 88.75 122.1)
 		(end 88.75 123.09)
@@
 	)
 	(segment
+		(start 93.4 109.95)
+		(end 93.7 110.25)
+		(width 0.2)
+		(layer "F.Cu")
+		(net 2)
+	)
+	(segment
 		(start 77.15 105.2)
 		(end 75.95 105.2)
@@
 	)
 	(segment
-		(start 92.1 110.03)
-		(end 92.1 110.45)
-		(width 0.2)
-		(layer "F.Cu")
-		(net 2)
-	)
-	(segment
 		(start 102.4 101.9)
 		(end 102.5 101.8)
@@
 	)
 	(segment
-		(start 92.1 110.45)
-		(end 92.6 110.95)
-		(width 0.2)
-		(layer "F.Cu")
-		(net 2)
-	)
-	(segment
 		(start 104.25 104.15)
 		(end 102.4 102.3)
@@
 	)
 	(segment
+		(start 92.6 109.95)
+		(end 93.4 109.95)
+		(width 0.2)
+		(layer "F.Cu")
+		(net 2)
+	)
+	(segment
 		(start 59.05 88.49)
 		(end 59.05 88.2)
@@
 	)
 	(segment
-		(start 98.8125 107.95)
-		(end 98.0625 107.2)
-		(width 0.2)
-		(layer "F.Cu")
-		(net 2)
-	)
-	(segment
 		(start 70 82.89)
 		(end 68.165 82.89)
@@
 	)
 	(via
-		(at 92.6 110.95)
+		(at 68.325 117.42)
 		(size 0.6)
 		(drill 0.3)
@@
 	)
 	(via
-		(at 68.325 117.42)
+		(at 65.174999 116.72)
 		(size 0.6)
 		(drill 0.3)
@@
 	)
 	(via
-		(at 65.174999 116.72)
+		(at 93.7 110.25)
 		(size 0.6)
 		(drill 0.3)
@@
 	)
 	(segment
+		(start 90.599 109.95)
+		(end 89.6 110.949)
+		(width 0.2)
+		(layer "F.Cu")
+		(net 4)
+	)
+	(segment
 		(start 72.3 115.34)
 		(end 73.55 116.59)
@@
 	)
 	(segment
+		(start 91.5 108.25)
+		(end 91.5 108.35)
+		(width 0.2)
+		(layer "F.Cu")
+		(net 4)
+	)
+	(segment
+		(start 90.7 109.15)
+		(end 90.7 109.95)
+		(width 0.2)
+		(layer "F.Cu")
+		(net 4)
+	)
+	(segment
 		(start 87.445 123.125)
 		(end 87.445 124.755)
@@
 	)
 	(segment
-		(start 91.5 108.47)
-		(end 92.1 109.07)
-		(width 0.2)
-		(layer "F.Cu")
-		(net 4)
-	)
-	(segment
 		(start 73.55 116.59)
 		(end 74.635 116.59)
@@
 	)
 	(segment
+		(start 91.5 108.35)
+		(end 90.7 109.15)
+		(width 0.2)
+		(layer "F.Cu")
+		(net 4)
+	)
+	(segment
 		(start 66.381499 115.345002)
 		(end 67.599998 115.345002)
@@
 	)
 	(segment
+		(start 90.7 109.95)
+		(end 90.599 109.95)
+		(width 0.2)
+		(layer "F.Cu")
+		(net 4)
+	)
+	(segment
 		(start 74.635 116.59)
 		(end 75.125 116.1)
@@
 	)
 	(via
+		(at 89.6 110.949)
+		(size 0.6)
+		(drill 0.3)
+		(layers "F.Cu" "B.Cu")
+		(net 4)
+	)
+	(via
 		(at 90.5 112.75)
 		(size 0.6)
@@
 	)
 	(segment
-		(start 91.15 108.25)
-		(end 90.5 108.9)
-		(width 0.2)
-		(layer "B.Cu")
-		(net 4)
-	)
-	(segment
 		(start 100.5 104.3)
 		(end 101.207109 105.007109)
@@
 	)
 	(segment
-		(start 91.5 108.25)
-		(end 91.15 108.25)
+		(start 90.5 111.849)
+		(end 90.5 112.75)
 		(width 0.2)
 		(layer "B.Cu")
@@
 	)
 	(segment
-		(start 90.5 108.9)
-		(end 90.5 112.75)
+		(start 89.6 110.949)
+		(end 90.5 111.849)
 		(width 0.2)
 		(layer "B.Cu")

Commit message: Generate new gerbers
Routing:
- net /UART1 RX: track 53.1 -> 51.3 mm
Changed lines of the file:
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@@
 			(usegerberattributes yes)
 			(usegerberadvancedattributes yes)
-			(creategerberjobfile yes)
+			(creategerberjobfile no)
 			(dashed_line_dash_ratio 12.000000)
 			(dashed_line_gap_ratio 3.000000)
@@
 	)
 	(segment
-		(start 98.750057 122.3)
+		(start 104.45 122.3)
+		(end 101.850057 122.3)
+		(width 0.2)
+		(layer "B.Cu")
+		(net 90)
+	)
+	(segment
+		(start 98.750057 119.2)
 		(end 98.750057 112.650057)
 		(width 0.2)
@@
 	)
 	(segment
-		(start 104.45 122.3)
-		(end 98.750057 122.3)
+		(start 98.750057 112.650057)
+		(end 94.149971 108.049971)
 		(width 0.2)
 		(layer "B.Cu")
@@
 	)
 	(segment
-		(start 98.750057 112.650057)
-		(end 94.149971 108.049971)
+		(start 94.3135 107.886443)
+		(end 94.3135 107.388557)
 		(width 0.2)
 		(layer "B.Cu")
@@
 	)
 	(segment
-		(start 94.3135 107.886443)
-		(end 94.3135 107.388557)
+		(start 101.850057 122.3)
+		(end 98.750057 119.2)
 		(width 0.2)
 		(layer "B.Cu")
